Commit message: Initiated Stoch in PyBullet

File: project_ws/stoch3/urdf/stoch3.urdf (robot description, URDF)
Before this commit: robot stoch3, 19 links, 18 joints
Links:
- removed link bl_foot_link
- removed link br_foot_link
- removed link fl_foot_link
- removed link fr_foot_link
- removed link world
- link base_link: geometry collision mesh filename=/home/swapnil/FoR_Project/project_ws/stoch3/meshes/base_lin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; visual mesh filename=/home/swapnil/FoR_Project/project_ws/stoch3/meshes/base_lin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
- link bl_abd_link: geometry collision mesh filename=/home/swapnil/FoR_Project/project_ws/stoch3/meshes/bl_abd_l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; visual mesh filename=/home/swapnil/FoR_Project/project_ws/stoch3/meshes/bl_abd_l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
- link bl_shank_link: geometry collision mesh filename=/home/swapnil/FoR_Project/project_ws/stoch3/meshes/bl_shank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; visual mesh filename=/home/swapnil/FoR_Project/project_ws/stoch3/meshes/bl_shank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
- link bl_thigh_link: geometry collision mesh filename=/home/swapnil/FoR_Project/project_ws/stoch3/meshes/bl_thigh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; visual mesh filename=/home/swapnil/FoR_Project/project_ws/stoch3/meshes/bl_thigh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
- link br_abd_link: geometry collision mesh filename=/home/swapnil/FoR_Project/project_ws/stoch3/meshes/br_abd_l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; visual mesh filename=/home/swapnil/FoR_Project/project_ws/stoch3/meshes/br_abd_l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
- link br_shank_link: geometry collision mesh filename=/home/swapnil/FoR_Project/project_ws/stoch3/meshes/br_shank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; visual mesh filename=/home/swapnil/FoR_Project/project_ws/stoch3/meshes/br_shank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
- link br_thigh_link: geometry collision mesh filename=/home/swapnil/FoR_Project/project_ws/stoch3/meshes/br_thigh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; visual mesh filename=/home/swapnil/FoR_Project/project_ws/stoch3/meshes/br_thigh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
- link fl_abd_link: geometry collision mesh filename=/home/swapnil/FoR_Project/project_ws/stoch3/meshes/fl_abd_l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; visual mesh filename=/home/swapnil/FoR_Project/project_ws/stoch3/meshes/fl_abd_l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
- link fl_shank_link: geometry collision mesh filename=/home/swapnil/FoR_Project/project_ws/stoch3/meshes/fl_shank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; visual mesh filename=/home/swapnil/FoR_Project/project_ws/stoch3/meshes/fl_shank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
- link fl_thigh_link: geometry collision mesh filename=/home/swapnil/FoR_Project/project_ws/stoch3/meshes/fl_thigh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; visual mesh filename=/home/swapnil/FoR_Project/project_ws/stoch3/meshes/fl_thigh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
- link fr_abd_link: geometry collision mesh filename=/home/swapnil/FoR_Project/project_ws/stoch3/meshes/fr_abd_l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; visual mesh filename=/home/swapnil/FoR_Project/project_ws/stoch3/meshes/fr_abd_l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
- link fr_shank_link: geometry collision mesh filename=/home/swapnil/FoR_Project/project_ws/stoch3/meshes/fr_shank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; visual mesh filename=/home/swapnil/FoR_Project/project_ws/stoch3/meshes/fr_shank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
- link fr_thigh_link: geometry collision mesh filename=/home/swapnil/FoR_Project/project_ws/stoch3/meshes/fr_thigh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; visual mesh filename=/home/swapnil/FoR_Project/project_ws/stoch3/meshes/fr_thigh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
Joints:
- removed joint bl_ankle_joint
- removed joint br_ankle_joint
- removed joint fl_ankle_joint
- removed joint fr_ankle_joint
- removed joint world_joint
